Commit message: Fix five real stability defects found by running the stack in Gazebo, and tell the truth about the sixth
Running the full stack end to end turned up defects that the wall-clock mode
never exposed. Each is individually justified, and each was verified before
moving on:

1. Floor markings had collision. Park pads are 2 cm boxes and the AGV spawns
   with its wheel bottoms at z=0.01, so every vehicle started 1 cm inside a pad:
   free to spin, unable to translate. All markings are now visual-only.
2. Dock slots had a physical can standing on the parking point, and the LiDAR
   emergency stop (0.38 m) is larger than the arrival tolerance (0.20 m), so a
   vehicle could never enter the point it was sent to. Cans live on the rack.
3. Arrival tolerance and emergency stop are now ordered correctly: inside 0.8 m
   of the target the LiDAR stop drops to 0.12 m (docking mode).
4. The LiDAR saw the vehicle's own front corners at 0.24 m inside its stop
   sector. Returns are now tested against the hull outline angle by angle.
   Non-zero velocity commands went from 0.5 % to 93 %.
5. Re-planning on a 3 s timer reset pure pursuit mid-turn and the vehicle
   oscillated in place. It now re-plans only when a peer occupies the next
   2.2 m of the path.

Also: wheel friction written as <mu1>/<mu2> does not survive URDF -> SDF
conversion in gz-sim (verified: zero <mu> in the output). The <surface> form
does, and is now used.

What is still broken is stated in the README rather than hidden: under Gazebo
the chassis does not reproduce commanded motion (0.17 m in 15 s at a held
0.5 m/s), so the wheel/ground contact model is not yet right. The coordination
stack commands correctly and the allocation result stands; the physical
repeatability does not yet.

READMEs: title centred, both condensed again (English 468 -> 290 lines), the
Andon board replaced by a still from the same renderer as the animation so the
two cannot drift apart, and a stability section added that says which parts are
measured and which are not.

File: src/fleetflow_sim/urdf/agv.urdf.xacro (robot description, xacro)
@@ -108,4 +108,6 @@
       <min_linear_acceleration>-2.5</min_linear_acceleration>
       <max_angular_acceleration>2.5</max_angular_acceleration>
+      <max_wheel_torque>20.0</max_wheel_torque>
+      <max_wheel_acceleration>8.0</max_wheel_acceleration>
       <!-- 话题必须按机器人加命名空间，否则多台车会共用 /odom /cmd_vel 互相串指令 -->
       <odom_topic>/robot_$(arg robot_id)/odom</odom_topic>
@@ -137,5 +139,29 @@
   </gazebo>
   <gazebo reference="base_link"><material>Gazebo/FlatBlack</material></gazebo>
-  <gazebo reference="left_wheel"><material>Gazebo/Black</material></gazebo>
-  <gazebo reference="right_wheel"><material>Gazebo/Black</material></gazebo>
+  <!-- 驱动轮接触参数：不写这些，圆柱轮与地面是线接触，默认摩擦下会明显打滑。
+       实测：指令 0.15 m/s 时 20 秒只走了 0.19 m（应走 3 m），差两个数量级，
+       整条线因此在 Gazebo 里几乎不产出。 -->
+  <gazebo reference="left_wheel">
+    <material>Gazebo/Black</material>
+    <surface>
+      <friction><ode><mu>1.8</mu><mu2>1.8</mu2></ode></friction>
+      <contact><ode><kp>1000000</kp><kd>100</kd><max_vel>0.1</max_vel><min_depth>0.001</min_depth></ode></contact>
+    </surface>
+  </gazebo>
+  <gazebo reference="right_wheel">
+    <material>Gazebo/Black</material>
+    <surface>
+      <friction><ode><mu>1.8</mu><mu2>1.8</mu2></ode></friction>
+      <contact><ode><kp>1000000</kp><kd>100</kd><max_vel>0.1</max_vel><min_depth>0.001</min_depth></ode></contact>
+    </surface>
+  </gazebo>
+  <!-- 万向轮是被动支撑，摩擦要低，否则会拖着车不让走 -->
+  <gazebo reference="caster">
+    <mu1>0.05</mu1><mu2>0.05</mu2>
+    <kp>1000000.0</kp><kd>100.0</kd>
+  </gazebo>
+  <!-- 车体不许蹭地 -->
+  <gazebo reference="base_link">
+    <mu1>0.02</mu1><mu2>0.02</mu2>
+  </gazebo>
 </robot>

Commit message: Make the traffic layer's collision criterion match the controller's
The ROS 1 traffic layer was ported with its original centre-distance
safety test: slow down inside 1.5 m, hard-stop inside 0.25 m. That test
was written for a 16x10 m layout with few robots. In this 26x16 m plant
eight AGVs are essentially always within 1.5 m of somebody, so the
coordinator pinned the whole fleet at speed_scale ~0.3 and never let go.

Meanwhile the controllers had already moved to an oriented-rectangle
(SAT) test in d0e2895. The two layers therefore disagreed about what
"about to collide" means. This makes the coordinator use the same
geometry: obb_gap() computes the gap between two hull outlines, and the
tier is now graded on that gap (slow below 0.45 m, stop below 0.06 m,
back off once the outlines actually overlap).

Measured on one machine in a single session:
  - median commanded speed 0.135 -> 0.150 m/s (cap is 0.85)
  - logic-mode "collision_slow" directives per 60 s: 1552 -> 238
  - Gazebo deliveries per 70 s with 8 robots: 0-2 -> 2-6

This is the only change this round whose effect survives the run-to-run
variance; see docs/gazebo-throughput-findings.md for the rest, including
the two claims in the handover that measurement disproved.

Also in this commit:

* metrics.py judged safety by centre distance with a 0.55 m "near miss"
  threshold, which is meaningless for 0.56x0.44 m hulls - two robots
  running side by side are legitimately 0.44 m apart. It now reports the
  outline gap and counts real overlaps: a run showing min_gap=0.10 m and
  overlap_events=0 is readable, whereas the old min_robot_distance_m=0.662
  was not. The old columns are kept so existing CSVs stay parseable.

* The start of the shift was a bottleneck in its own right: eight robots
  parked 1.35 m apart all set off together and jammed. start_stagger
  releases robot i after i*stagger seconds, which took 8 robots from
  0 to 3.4 deliveries/min. Fleet scaling is otherwise linear - 2 robots
  manage 3.0/min and 4 manage 6.0/min - so the collapse was in the
  departure, not the coordination.

* Debug switches (debug_avoid, debug_scan_dir, avoid_cones) default off
  and exist so the next person can re-run the investigations documented
  in docs/ without re-deriving them.

File: src/fleetflow_sim/urdf/agv.urdf.xacro (robot description, xacro)
@@ -122,5 +122,5 @@
     <sensor name="lidar" type="gpu_lidar">
       <topic>/robot_$(arg robot_id)/scan</topic>
-      <update_rate>8</update_rate>
+      <update_rate>8.0</update_rate>
       <always_on>1</always_on>
       <visualize>false</visualize>
@@ -139,21 +139,16 @@
   </gazebo>
   <gazebo reference="base_link"><material>Gazebo/FlatBlack</material></gazebo>
-  <!-- 驱动轮接触参数：不写这些，圆柱轮与地面是线接触，默认摩擦下会明显打滑。
-       实测：指令 0.15 m/s 时 20 秒只走了 0.19 m（应走 3 m），差两个数量级，
-       整条线因此在 Gazebo 里几乎不产出。 -->
-  <gazebo reference="left_wheel">
-    <material>Gazebo/Black</material>
-    <surface>
-      <friction><ode><mu>1.8</mu><mu2>1.8</mu2></ode></friction>
-      <contact><ode><kp>1000000</kp><kd>100</kd><max_vel>0.1</max_vel><min_depth>0.001</min_depth></ode></contact>
-    </surface>
-  </gazebo>
-  <gazebo reference="right_wheel">
-    <material>Gazebo/Black</material>
-    <surface>
-      <friction><ode><mu>1.8</mu><mu2>1.8</mu2></ode></friction>
-      <contact><ode><kp>1000000</kp><kd>100</kd><max_vel>0.1</max_vel><min_depth>0.001</min_depth></ode></contact>
-    </surface>
-  </gazebo>
+  <gazebo reference="left_wheel"><material>Gazebo/Black</material></gazebo>
+  <gazebo reference="right_wheel"><material>Gazebo/Black</material></gazebo>
+  <!-- 摩擦系数在这里**写不进去**，留个记录免得再试一遍：
+       sdformat 的 URDF 解析器会把摩擦信息整段丢掉 —— 无论是
+       <gazebo reference="link"><mu1>/<mu2>，还是 <collision> 里的
+       <surface><friction>，转换后都**不出现**在 SDF 里，而且不报错。
+       验证方法：gz sdf -p 转一个最小 URDF，输出里既没有 <surface>
+       也没有 <mu>。所以轮子只能拿 SDF 默认摩擦（1.0）。
+       这也说明"轮子打滑"不是厂房里那台车不走的根因 —— 作为对照，
+       把同一台车放进只有一块平地的最小世界，用 gz 原生话题发 0.6 m/s，
+       7 秒实走 3.57 m（≈0.6 m/s），轮速恰好 8.000 rad/s，完全正常。
+       真正的排查结论见 tools/ 与 README 的"排查记录"。 -->
   <!-- 万向轮是被动支撑，摩擦要低，否则会拖着车不让走 -->
   <gazebo reference="caster">

Commit message: Rebuild at industrial scale: 120x60 m plant, 50 cm circular AGVs, 6:6:6 stations
You were right on all three counts, and checking the previous FleetFlow repo confirmed the
mechanism. That plant was 12x10 m with 0.075x0.0875 m robots - symbol-sized. Ten of them did not
deadlock because each was almost nothing relative to the aisle. The intermediate version here
had 0.56x0.44 m robots in 0.65 m aisles, which is why it locked up, and 32x16 m is not a
realistic mill footprint either.

layout.py now carries the industrial scale: a 120x60 m hall, an AGV spec of 0.50 m diameter,
0.30 m height, 0.36 m wheelbase and a 12 m lidar, and named constants AISLE=3.0, LANE_PITCH=3.0
and LANES_PER_STAGE=6 so the tightness is one number rather than scattered literals. Stage
geometry is regrouped to 15 m per stage with 9.2 m between stages, six docking slots per store
aligned with the production lanes, and the park lane moved to the south wall. The URDF body is a
cylinder now with a round deck, a heading marker and a 360-degree lidar at 360 samples.

traffic.py follows the circular geometry: a new circle_gap() computes centre distance minus two
radii, and the entire oriented-bounding-box and separating-axis implementation is deleted,
because a circle's footprint does not depend on heading and that code had itself become a source
of bugs. Safety thresholds are recalibrated for the larger vehicle - slow at 0.60 m, hard stop at
0.10 m, overlap at 0 m. Region definitions are derived from the layout instead of hard-coded.

The one-way corridor tokens are switched off. Their premise was an aisle that fits barely one
vehicle; the new inter-stage clearance is 9.2 m, eleven times the 0.80 m passing requirement, so
the tokens could only manufacture waiting. CORRIDOR_ZONES is empty and the code path remains for
reinstatement.

One real bug surfaced while testing. _true_speed_now() used pose differencing alone when no
odometry is available, but in logic mode the pose updates in bursts, so the difference reads zero
for most control cycles. The coordinator then concluded the vehicle was stopped and fired
stalled_replan every 8 s at robots that were driving normally - all four triggered within 45 s.
It now takes the larger of the pose difference and the commanded speed: the command is non-zero
while the vehicle is genuinely moving, and zero when it is genuinely stopped, so the maximum
cannot turn a stop into motion. False stalls went from 15 to zero.

Measured after the change, six AGVs over 260 s in logic mode: median dwell is 27.5 s to pickup,
17.2 s to dropoff, 1.3 s departing, 1.2 s loading and 0.11 s waiting for a lease. Travel
dominates because a single leg is now 25 to 47 m; leases, handling and avoidance are no longer
bottlenecks. Longer legs and a slower cadence are the inherent cost of the larger plant, and the
compensating levers are fleet size and per-stage buffering rather than avoidance tuning.

File: src/fleetflow_sim/urdf/agv.urdf.xacro (robot description, xacro)
@@ -6,12 +6,14 @@
   <xacro:property name="robot_id"   value="$(arg robot_id)"/>
   <xacro:property name="body_color" value="$(arg body_color)"/>
-  <!-- 尺寸: 一台能放进 16x10m 厂房、又能在截图里看清的搬运车 -->
-  <xacro:property name="body_len" value="0.56"/>
-  <xacro:property name="body_w"   value="0.44"/>
-  <xacro:property name="body_h"   value="0.14"/>
-  <xacro:property name="wheel_r"  value="0.075"/>
-  <xacro:property name="wheel_w"  value="0.045"/>
-  <xacro:property name="sep"      value="0.42"/>
-  <xacro:property name="deck_z"   value="${body_h/2 + 0.02}"/>
+  <!-- 尺寸：**直径 0.50 m 的圆盘差速底盘**（layout.AGV 是同一份规格）。
+       工业 AGV 多用圆车：任意朝向占地相同，避让判据不必分朝向。
+       参数取公开规格的量级（松灵/宇树这类底盘：直径 0.4~0.6 m、
+       高 0.25~0.35 m、轮距约 0.36 m、带 360° 雷达）。 -->
+  <xacro:property name="body_r"   value="0.25"/>   <!-- 半径 = 直径 0.50 -->
+  <xacro:property name="body_h"   value="0.24"/>
+  <xacro:property name="wheel_r"  value="0.06"/>
+  <xacro:property name="wheel_w"  value="0.04"/>
+  <xacro:property name="sep"      value="0.36"/>   <!-- 轮距（左右轮中心距） -->
+  <xacro:property name="deck_z"   value="${body_h/2 + 0.012}"/>
   <link name="base_footprint"/>
   <joint name="base_joint" type="fixed">
@@ -22,21 +24,27 @@
   <link name="base_link">
     <visual name="body">
-      <geometry><box size="${body_len} ${body_w} ${body_h}"/></geometry>
+      <geometry><cylinder radius="${body_r}" length="${body_h}"/></geometry>
       <material name="body"><color rgba="${body_color} 1"/></material>
     </visual>
-    <!-- 顶面浅色甲板，俯视时能一眼分清车体和朝向 -->
+    <!-- 顶面浅色甲板（圆），俯视时能一眼分清车体 -->
     <visual name="deck">
-      <origin xyz="-0.06 0 ${deck_z}" rpy="0 0 0"/>
-      <geometry><box size="0.30 0.30 0.02"/></geometry>
+      <origin xyz="0 0 ${deck_z}" rpy="0 0 0"/>
+      <geometry><cylinder radius="${body_r*0.78}" length="0.012"/></geometry>
       <material name="deck"><color rgba="0.96 0.97 0.98 1"/></material>
     </visual>
-    <!-- 车头标记，用于判断朝向 -->
+    <!-- 车头指向标记：俯视时的朝向全靠它 -->
     <visual name="nose">
-      <origin xyz="${body_len/2 - 0.03} 0 0.01" rpy="0 0 0"/>
-      <geometry><box size="0.06 0.20 0.04"/></geometry>
+      <origin xyz="${body_r*0.72} 0 ${body_h/2 - 0.005}" rpy="0 0 0"/>
+      <geometry><box size="0.10 0.06 0.02"/></geometry>
       <material name="nose"><color rgba="1.0 0.45 0.10 1"/></material>
     </visual>
+    <!-- 360° 雷达（顶部圆柱），与 LiDAR 安装高度一致 -->
+    <visual name="lidar">
+      <origin xyz="${body_r*0.55} 0 ${body_h/2 + 0.03}" rpy="0 0 0"/>
+      <geometry><cylinder radius="0.035" length="0.05"/></geometry>
+      <material name="lidar"><color rgba="0.12 0.12 0.14 1"/></material>
+    </visual>
     <collision name="body_c">
-      <geometry><box size="${body_len} ${body_w} ${body_h}"/></geometry>
+      <geometry><cylinder radius="${body_r}" length="${body_h}"/></geometry>
     </collision>
     <inertial>
@@ -86,5 +94,5 @@
     <parent link="base_link"/>
     <child link="caster"/>
-    <origin xyz="${-body_len/2 + 0.06} 0 ${-body_h/2 - 0.03}" rpy="0 0 0"/>
+    <origin xyz="${-body_r*0.72} 0 ${-body_h/2 - 0.03}" rpy="0 0 0"/>
   </joint>
   <link name="lidar_link">
@@ -96,5 +104,5 @@
     <parent link="base_link"/>
     <child link="lidar_link"/>
-    <origin xyz="${body_len/2 - 0.10} 0 ${body_h/2 + 0.045}" rpy="0 0 0"/>
+    <origin xyz="0 0 ${body_h/2 + 0.045}" rpy="0 0 0"/>
   </joint>
   <!-- ============ Gazebo Sim 系统 ============ -->
@@ -128,5 +136,5 @@
         <scan>
           <horizontal>
-            <samples>180</samples>
+            <samples>360</samples>
             <resolution>1</resolution>
             <min_angle>-3.14159</min_angle>
@@ -135,4 +143,5 @@
         </scan>
         <range><min>0.12</min><max>12.0</max><resolution>0.01</resolution></range>
+        <!-- 量程 12 m 与 layout.AGV['lidar_range'] 一致：主通道 9.2 m 内可全见 -->
       </lidar>
     </sensor>
